File: SCH-PCB/arcadeController/EAGLE/arcadeController.sch (EAGLE design)
At the start: 26 parts, among them J2 1759046, J3 1759046, J4 1759046, J5 1759046, U1 RASPBERRY_PICOSMD-TH, X1 04-JST-B4B-XH-A, X2 04-JST-B4B-XH-A, X3 04-JST-B4B-XH-A, X4 04-JST-B4B-XH-A, X5 04-JST-B4B-XH-A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

Commit message: FIX: PCB design there are line with <0.1mm
Other:
- note removed: "ARCADE CONTROLLER RP2040"
- note removed: "BOLT HOLE"
- note removed: "CONNECTOR JST-XH"
- note removed: "Juarendra Ramadhani"
- note removed: "LED RGB"
- note removed: "MALE HEADER"
- note removed: "Microcontroller"
- note removed: "PLUGABLE CONNECTOR"
- note removed: "PULLUP I2C"
- moved on the sheet: C1, LED1, R1, R2, R3, R4, R5, R6, U1, X1-1, X1-2, X1-3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
